File: amigaypbpr.kicad_pcb (KiCad board)
At the start: 2 copper layers, 28 x 49 mm, 26 parts, among them J1 DB25_Female, J2 PB, J3 PR, U1 OPA2356xxD, U2 OPA2356xxD, U3 OPA2356xxD

Commit message: pin assignments
Other:
- net class Default removed
